Commit message: Robot fisico: launch sin Gazebo, firmware ESP32, scripts de prueba y notas
- champ_real.launch.py + gait_real.yaml: CHAMP sin Gazebo para el robot real.
- Puentes ROS2: joint_trajectory_bridge.py (CHAMP -> ESP32) e imu_publisher.py.
- hardware/esp32_firmware: sketch del bridge (1 PCA9685, calibracion 25 sept)
  y sketches de calibracion/escaner I2C.
- hardware/scripts_pruebas: creep_una_pata.py (marcha creep con desplazamiento
  de peso) y prueba_dos_patas.py.
- Mundo turtlebot3 pequeno + launches slam/amcl_pequeno y mapa_chico.
- URDF: shift (coxa->femur) corregido a 0.043 m.
- CLAUDE.md: notas de calibracion, hardware y lecciones aprendidas.

Co-Authored-By: Claude Sonnet 5 <noreply@anthropic.com>
Claude-Session: https://claude.ai/code/session_01PZ78r6NaVpjvzekwDHAwZD

File: src/robot_dog/urdf/spot_micro.urdf.xacro (robot description, xacro)
@@ -26,5 +26,5 @@
   <xacro:property name="toe_radius" value="0.020" />
   <xacro:property name="toe_width" value="0.020" />
-  <xacro:property name="shift" value="0.055" />
+  <xacro:property name="shift" value="0.043" />
   <xacro:property name="shiftx" value="0.093" />
   <xacro:property name="shifty" value="0.039" />
@@ -215,5 +215,5 @@
     <parent link="base_footprint"/>
     <child link="base_link"/>
-    <origin xyz="0 0 0.26" rpy="0 0 0"/>
+    <origin xyz="0 0 0.15" rpy="0 0 0"/>
   </joint>
   <link name="base_link">
